File: PCB/3DWelderPCB.kicad_pcb (KiCad board)
At the start: 2 copper layers, 31.8 x 114.8 mm, 17 parts, among them J1 0.91in OLED Display, J2 Screw_Terminal_01x04 IN, J4 24V Fan, J5 Thermistor, J6 Screw_Terminal_01x02, Q2 IRLZ34N, SW1 EC11 RotaryEncoder_Switch

Commit message: PCBV3
Parts:
- R1: value R100k -> 4.7K
- moved R2 26.2 mm to (145.7, 86.8)
- moved R5 22.5 mm to (142.4, 86.8)
- moved J1 0.22 mm to (129.2, 122.9)
Connections:
- net /Heater GND renamed Heater GND
- net /Thermistor renamed Thermistor
- A1 pad 10: /EC11SWB -> unconnected-(A1-D7-Pad10)
- A1 pad 23: Net-(A1-A4) -> SDA
- A1 pad 24: Net-(A1-A5) -> SCL
- A1 pad 5: unconnected-(A1-D2-Pad5) -> EC11A
- A1 pad 6: /Heater -> EC11B
- A1 pad 7: /EC11B -> Heater
- A1 pad 8: /EC11A -> EC11SWA
- A1 pad 9: /EC11SWA -> EC11SWB
- J1 pad 1: /SDA -> GND
- J1 pad 2: /SCL -> +5V
- J1 pad 3: +5V -> SCL
- J1 pad 4: GND -> SDA
- R2 pad 1: Net-(A1-A4) -> SCL
- R2 pad 2: /SDA -> +5V
- R4 pad 1: /Heater -> Heater
- R5 pad 1: Net-(A1-A5) -> SDA
- R5 pad 2: /SCL -> +5V
- SW1 pad A: /EC11A -> EC11A
- SW1 pad B: /EC11B -> EC11B
- SW1 pad S1: /EC11SWA -> EC11SWA
- SW1 pad S2: /EC11SWB -> EC11SWB
Routing:
- net /EC11A: track 84.4 -> 0.00 mm
- net EC11A: track 0.00 -> 81.9 mm
- net /EC11B: track 79.8 -> 0.00 mm
- net EC11B: track 0.00 -> 77.2 mm
- net /EC11SWB: track 75.0 -> 0.00 mm
- net EC11SWB: track 0.00 -> 72.4 mm
- net /EC11SWA: track 70.4 -> 0.00 mm
- net EC11SWA: track 0.00 -> 67.8 mm
- net SCL: track 0.00 -> 32.9 mm, vias 0 -> 1
- net /SDA: track 31.2 -> 0.00 mm, vias 2 -> 0
- net SDA: track 0.00 -> 28.5 mm, vias 0 -> 1
- net /SCL: track 23.2 -> 0.00 mm, vias 1 -> 0
- net Heater: track 0.00 -> 14.2 mm
- net /Heater: track 11.6 -> 0.00 mm
- net +5V: track 45.3 -> 49.5 mm
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