File: PCB/3DWelderSchematic.kicad_sch (KiCad schematic)
At the start: 13 parts, among them J1 0.91in OLED Display, J2 Screw_Terminal_01x04 IN, J4 24V Fan, J5 Thermistor, J6 Screw_Terminal_01x02, Q2 IRLZ34N, SW1 EC11 RotaryEncoder_Switch

Commit message: PCBV3
Parts:
- R1: value R100k -> 4.7K
Connections:
- net +5V: now also J1.2 (Pin_2), R2.2, R5.2; no longer J1.3 (Pin_3)
- net EC11A: now also A1.5 (D2); no longer A1.8 (D5)
- net EC11B: now also A1.6 (D3); no longer A1.7 (D4)
- net EC11SWA: now also A1.8 (D5); no longer A1.9 (D6)
- net EC11SWB: now also A1.9 (D6); no longer A1.10 (D7)
- net GND: now also J1.1 (Pin_1); no longer J1.4 (Pin_4)
- net Heater: now also A1.7 (D4); no longer A1.6 (D3)
- net SCL: now also A1.24 (A5), J1.3 (Pin_3), R2.1; no longer J1.2 (Pin_2), R5.2
- net SDA: now also A1.23 (A4), J1.4 (Pin_4), R5.1; no longer J1.1 (Pin_1), R2.2
Other:
- moved on the sheet: J1, R2, R5
